Commit message: Initial URDF done working

File: install/homebot/share/homebot/urdf/homebot_core.xacro (robot description, xacro)
@@ -1,4 +1,6 @@
 <?xml version="1.0"?>
 <robot xmlns:xacro="http://www.ros.org/wiki/xacro">
+    <xacro:include filename="inertial_macros.xacro" />
+    <!-- Colors  -->
     <material name="black">
         <color rgba="0 0 0 1"/>
@@ -13,6 +15,11 @@
         <color rgba="0 1 0 1"/>
     </material>
+    <material name="grey">
+        <color rgba="0.5 0.5 0.5 1"/>
+    </material>
+    <!-- Base Link  -->
     <link name="base_link">
     </link>
+    <!-- Chassis Joint  -->
     <joint name="chassis_joint" type="fixed">
         <origin xyz="-0.1 0 0" rpy="0 0 0"/>
@@ -20,4 +27,5 @@
         <child link="chassis"/>
     </joint>
+    <!-- Chassis Link  -->
     <link name="chassis">
         <visual>
@@ -34,4 +42,84 @@
             </geometry>
         </collision>
+        <inertial_box mass="0.5" x="0.3" y="0.3" z="0.15">
+            <origin xyz="0.15 0 0.075" rpy="0 0 0"/>
+        </inertial_box>
     </link>
+    <!-- Left Wheel Joint  -->
+    <joint name="left_wheel_joint" type="continuous">
+        <origin xyz="0 0.175 0" rpy="-${pi/2} 0 0"/>
+        <parent link="base_link"/>
+        <child link="left_wheel"/>
+        <axis xyz="0 0 1"/>
+    </joint>
+    <!-- Left Wheel Link  -->
+    <link name="left_wheel">
+        <visual>
+            <origin xyz="0 0 0" rpy="0 0 0"/>
+            <geometry>
+                <cylinder radius="0.05" length="0.05"/>
+            </geometry>
+            <material name="black"/>
+        </visual>
+        <collision>
+            <origin xyz="0 0 0" rpy="0 0 0"/>
+            <geometry>
+                <cylinder radius="0.05" length="0.05"/>
+            </geometry>
+        </collision>
+        <inertial_cylinder mass="0.1" length="0.05" radius="0.05">
+            <origin xyz="0 0 0" rpy="0 0 0"/>
+        </inertial_cylinder>
+    </link>
+    <!-- Right Wheel Joint  -->
+    <joint name="right_wheel_joint" type="continuous">
+        <origin xyz="0 -0.175 0" rpy="${pi/2} 0 0"/>
+        <parent link="base_link"/>
+        <child link="right_wheel"/>
+        <axis xyz="0 0 -1"/>
+    </joint>
+    <!-- Right Wheel Link  -->
+    <link name="right_wheel">
+        <visual>
+            <origin xyz="0 0 0" rpy="0 0 0"/>
+            <geometry>
+                <cylinder radius="0.05" length="0.05"/>
+            </geometry>
+            <material name="black"/>
+        </visual>
+        <collision>
+            <origin xyz="0 0 0" rpy="0 0 0"/>
+            <geometry>
+                <cylinder radius="0.05" length="0.05"/>
+            </geometry>
+        </collision>
+        <inertial_cylinder mass="0.1" length="0.05" radius="0.05">
+            <origin xyz="0 0 0" rpy="0 0 0"/>
+        </inertial_cylinder>
+    </link>
+    <!-- Castor Link  -->
+    <link name="castor">
+        <visual>
+            <origin xyz="0 0 0" rpy="0 0 0"/>
+            <geometry>
+                <sphere radius="0.025"/>
+            </geometry>
+            <material name="grey"/>
+        </visual>
+        <collision>
+            <origin xyz="0 0 0" rpy="0 0 0"/>
+            <geometry>
+                <sphere radius="0.025"/>
+            </geometry>
+        </collision>
+        <inertial_sphere mass="0.1" radius="0.025">
+            <origin xyz="0 0 0" rpy="0 0 0"/>
+        </inertial_sphere>
+    </link>
+    <!-- Castor Joint  -->
+    <joint name="castor_joint" type="fixed">
+        <origin xyz="0.175 0 -0.025" rpy="0 0 0"/>
+        <parent link="base_link"/>
+        <child link="castor"/>
+    </joint>
 </robot>

Commit message: Fixed launch file bug where JSP didnt work correct

File: install/homebot/share/homebot/urdf/homebot_core.xacro (robot description, xacro)
@@ -1,5 +1,4 @@
 <?xml version="1.0"?>
 <robot xmlns:xacro="http://www.ros.org/wiki/xacro">
-    <xacro:include filename="inertial_macros.xacro" />
     <!-- Colors  -->
     <material name="black">
@@ -42,7 +41,4 @@
             </geometry>
         </collision>
-        <inertial_box mass="0.5" x="0.3" y="0.3" z="0.15">
-            <origin xyz="0.15 0 0.075" rpy="0 0 0"/>
-        </inertial_box>
     </link>
     <!-- Left Wheel Joint  -->
@@ -68,7 +64,4 @@
             </geometry>
         </collision>
-        <inertial_cylinder mass="0.1" length="0.05" radius="0.05">
-            <origin xyz="0 0 0" rpy="0 0 0"/>
-        </inertial_cylinder>
     </link>
     <!-- Right Wheel Joint  -->
@@ -94,7 +87,4 @@
             </geometry>
         </collision>
-        <inertial_cylinder mass="0.1" length="0.05" radius="0.05">
-            <origin xyz="0 0 0" rpy="0 0 0"/>
-        </inertial_cylinder>
     </link>
     <!-- Castor Link  -->
@@ -113,7 +103,4 @@
             </geometry>
         </collision>
-        <inertial_sphere mass="0.1" radius="0.025">
-            <origin xyz="0 0 0" rpy="0 0 0"/>
-        </inertial_sphere>
     </link>
     <!-- Castor Joint  -->

File: src/homebot/urdf/inertial_macros.xacro (robot description, xacro)
@@ -1,5 +1,4 @@
-<!-- Copied from https://github.com/joshnewans/articubot_one/blob/d5aa5e9bc9039073c0d8fd7fe426e170be79c087/description/inertial_macros.xacro -->
 <?xml version="1.0"?>
-<robot xmlns:xacro="http://www.ros.org/wiki/xacro" >
+<robot xmlns:xacro="http://www.ros.org/wiki/xacro">
     <!-- Specify some standard inertial calculations https://en.wikipedia.org/wiki/List_of_moments_of_inertia -->
     <!-- These make use of xacro's mathematical functionality -->

Commit message: Made xacro properties for robot physical parameters and added interia

File: install/homebot/share/homebot/urdf/homebot_core.xacro (robot description, xacro)
@@ -1,4 +1,24 @@
 <?xml version="1.0"?>
 <robot xmlns:xacro="http://www.ros.org/wiki/xacro">
+    <!-- Import inertial macros -->
+    <xacro:include filename="inertial_macros.xacro"/>
+    <!-- Physical Parameters -->
+    <xacro:property name="wheel_radius" value="0.05"/>
+    <xacro:property name="wheel_width" value="0.05"/>
+    <xacro:property name="castor_radius" value="${wheel_radius/2}"/>
+    <xacro:property name="chassis_y_len" value="0.3"/>
+    <xacro:property name="chassis_x_len" value="0.3"/>
+    <xacro:property name="chassis_z_len" value="0.15"/>
+    <xacro:property name="wheel_mass" value="0.1"/>
+    <xacro:property name="chassis_mass" value="0.5"/>
+    <xacro:property name="castor_mass" value="0.1"/>
+    <!-- Castor offset from chassis link -->
+    <xacro:property name="castor_x" value="${chassis_x_len - chassis_x_len/7}"/>
+    <xacro:property name="castor_y" value="0"/>
+    <xacro:property name="castor_z" value="-${castor_radius}"/>
+    <!-- Chassis offset from base link -->
+    <xacro:property name="chassis_x" value="-0.1"/>
+    <xacro:property name="chassis_y" value="0"/>
+    <xacro:property name="chassis_z" value="0"/>
     <!-- Colors  -->
     <material name="black">
@@ -17,4 +37,7 @@
         <color rgba="0.5 0.5 0.5 1"/>
     </material>
+    <material name="blue">
+        <color rgba="0 0 1 0.7"/>
+    </material>
     <!-- Base Link  -->
     <link name="base_link">
@@ -22,5 +45,5 @@
     <!-- Chassis Joint  -->
     <joint name="chassis_joint" type="fixed">
-        <origin xyz="-0.1 0 0" rpy="0 0 0"/>
+        <origin xyz="${chassis_x} ${chassis_y} ${chassis_z}" rpy="0 0 0"/>
         <parent link="base_link"/>
         <child link="chassis"/>
@@ -29,20 +52,23 @@
     <link name="chassis">
         <visual>
-            <origin xyz="0.15 0 0.075" rpy="0 0 0"/>
+            <origin xyz="${chassis_x_len/2} 0 ${chassis_z_len/2}" rpy="0 0 0"/>
             <geometry>
-                <box size="0.3 0.3 0.15"/>
+                <box size="${chassis_x_len} ${chassis_y_len} ${chassis_z_len}"/>
             </geometry>
-            <material name="green"/>
+            <material name="blue"/>
         </visual>
         <collision>
-            <origin xyz="0 0 0" rpy="0 0 0"/>
+            <origin xyz="${chassis_x_len/2} 0 ${chassis_z_len/2}" rpy="0 0 0"/>
             <geometry>
-                <box size="0.3 0.3 0.15"/>
+                <box size="${chassis_x_len} ${chassis_y_len} ${chassis_z_len}"/>
             </geometry>
         </collision>
+        <xacro:inertial_box mass="${chassis_mass}" x="${chassis_x_len}" y="${chassis_y_len}" z="${chassis_z_len}">
+            <origin xyz="${chassis_x_len/2} 0 ${chassis_z_len/2}" rpy="0 0 0"/>
+        </xacro:inertial_box>
     </link>
     <!-- Left Wheel Joint  -->
     <joint name="left_wheel_joint" type="continuous">
-        <origin xyz="0 0.175 0" rpy="-${pi/2} 0 0"/>
+        <origin xyz="0 ${chassis_y_len/2 + wheel_width/2} 0" rpy="-${pi/2} 0 0"/>
         <parent link="base_link"/>
         <child link="left_wheel"/>
@@ -54,5 +80,5 @@
             <origin xyz="0 0 0" rpy="0 0 0"/>
             <geometry>
-                <cylinder radius="0.05" length="0.05"/>
+                <cylinder radius="${wheel_radius}" length="${wheel_width}"/>
             </geometry>
             <material name="black"/>
@@ -61,11 +87,14 @@
             <origin xyz="0 0 0" rpy="0 0 0"/>
             <geometry>
-                <cylinder radius="0.05" length="0.05"/>
+                <cylinder radius="${wheel_radius}" length="${wheel_width}"/>
             </geometry>
         </collision>
+        <xacro:inertial_cylinder mass="${wheel_mass}" length="${wheel_width}" radius="${wheel_radius}">
+            <origin xyz="0 0 0" rpy="0 0 0"/>
+        </xacro:inertial_cylinder>
     </link>
     <!-- Right Wheel Joint  -->
     <joint name="right_wheel_joint" type="continuous">
-        <origin xyz="0 -0.175 0" rpy="${pi/2} 0 0"/>
+        <origin xyz="0 -${chassis_y_len/2 + wheel_width/2} 0" rpy="${pi/2} 0 0"/>
         <parent link="base_link"/>
         <child link="right_wheel"/>
@@ -77,5 +106,5 @@
             <origin xyz="0 0 0" rpy="0 0 0"/>
             <geometry>
-                <cylinder radius="0.05" length="0.05"/>
+                <cylinder radius="${wheel_radius}" length="${wheel_width}"/>
             </geometry>
             <material name="black"/>
@@ -84,8 +113,17 @@
             <origin xyz="0 0 0" rpy="0 0 0"/>
             <geometry>
-                <cylinder radius="0.05" length="0.05"/>
+                <cylinder radius="${wheel_radius}" length="${wheel_width}"/>
             </geometry>
         </collision>
+        <xacro:inertial_cylinder mass="${wheel_mass}" length="${wheel_width}" radius="${wheel_radius}">
+            <origin xyz="0 0 0" rpy="0 0 0"/>
+        </xacro:inertial_cylinder>
     </link>
+    <!-- Castor Joint  -->
+    <joint name="castor_joint" type="fixed">
+        <origin xyz="${castor_x} ${castor_y} ${castor_z}" rpy="0 0 0"/>
+        <parent link="chassis"/>
+        <child link="castor"/>
+    </joint>
     <!-- Castor Link  -->
     <link name="castor">
@@ -93,5 +131,5 @@
             <origin xyz="0 0 0" rpy="0 0 0"/>
             <geometry>
-                <sphere radius="0.025"/>
+                <sphere radius="${castor_radius}"/>
             </geometry>
             <material name="grey"/>
@@ -100,13 +138,10 @@
             <origin xyz="0 0 0" rpy="0 0 0"/>
             <geometry>
-                <sphere radius="0.025"/>
+                <sphere radius="${castor_radius}"/>
             </geometry>
         </collision>
+        <xacro:inertial_sphere mass="${castor_mass}" radius="${castor_radius}">
+            <origin xyz="0 0 0" rpy="0 0 0"/>
+        </xacro:inertial_sphere>
     </link>
-    <!-- Castor Joint  -->
-    <joint name="castor_joint" type="fixed">
-        <origin xyz="0.175 0 -0.025" rpy="0 0 0"/>
-        <parent link="base_link"/>
-        <child link="castor"/>
-    </joint>
 </robot>
